File: schematic/logic.sch (KiCad schematic (older format))
At the start: 69 parts

Commit message: new headers files
Parts:
- removed P?: CONN_1, symbol CONN_1
- removed R?: 10K, symbol R
- added C10, C9: CP, symbol CP
- added D22, D5: LED, symbol LED
- added IC3, IC4: 74LS14N, 74xx-eu-DIL14, symbol 74LS14N
- added R10, R13: 2K2, symbol R
- added R11, R30: 58K, symbol R
- added R12, R31: 330, symbol R
- added SW2, SW3: SW_PUSH, symbol SW_PUSH
- gave numbers to parts that had none: 67
Connections:
- net +5V: now also R11.2, R30.2
- net GND: now also U1.23 (BLANK), D22.2 (K), D5.2 (K), SW2.2, SW3.2
- net at IC1.18 ((PCINT4/MISO)PB4), P1.1: now also R9.2
- net at IC1.24 ((PCINT9/ADC1)PC1): now also IC2.6 (O)
- net at IC1.25 ((PCINT10/ADC2)PC2): now also IC4.6 (O)
- net at IC1.26 ((PCINT11/ADC3)PC3): now also IC3.6 (O)
- net at IC1.28 ((PCINT14/SCL/ADC5)PC5): now also R12.2; no longer U1.23 (BLANK)
- net at IC1.3 ((PCINT17/TXD)PD1), P2.2: now also R31.2
- new net: R13.1, R30.1, SW3.1
- new net: D22.1 (A), R31.1
- new net: C10.1, IC4.5 (I), R13.2
- new net: R10.1, R11.1, SW2.1
- new net: C9.1, IC3.5 (I), R10.2
- new net: D5.1 (A), R12.1
Other:
- note added: "BUS\nPush Buttons\n"
- note added: "From Voice Rec.\nRx Input"
- note removed: "BUS\nPush Button\n"
- note removed: "Serial\nTo Voice Rec."
- moved on the sheet: C5, C6, C7, C8, D1, D2, D3, IC2F, P1, P3, P4, P5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
